File: RC_CAR_V3/rc_car_v3.brd (EAGLE design)
At the start: 80 x 68 mm, 60 parts, among them IC1 LIS2DW12TR, IC2 INA199B3DCKR, IC4 CY8C5888LTI-LP097, J1 282836-2, J2 282836-2, J3 1-1734742-8, J4 282836-2, Q1 2N7002-7-F, Q2 2N7002-7-F, Q5 SQJ912AEP-T2_BE3, Q7 SI7923DN-T1-E3, U1 MCP1703T-3302E/DB

Commit message: Changes
Changed lines of the file:
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@@
 <vertex x="63.754" y="84.836" curve="-90"/>
 <vertex x="61.849" y="82.931"/>
-<vertex x="49.657" y="82.931"/>
 <vertex x="40.386" y="82.931" curve="90"/>
 <vertex x="38.735" y="81.28"/>
@@
 <vertex x="88.646" y="28.829" curve="90"/>
 <vertex x="89.916" y="30.099"/>
-<vertex x="89.916" y="88.773" curve="90"/>
-<vertex x="88.519" y="90.17"/>
-<vertex x="64.897" y="90.17" curve="90"/>
-<vertex x="63.754" y="89.027"/>
+<vertex x="89.916" y="84.836"/>
 </polygon>
 <via x="65.151" y="83.82" extent="1-16" drill="0.35"/>
@@
 <vertex x="31.369" y="29.083" curve="-90"/>
 </polygon>
+<via x="64.389" y="66.167" extent="1-16" drill="0.35"/>
 <wire x1="38.862" y1="66.003" x2="42.734" y2="66.294" width="0" layer="19" extent="1-1"/>
-<wire x1="63.438" y1="69.342" x2="54.178" y2="70.244" width="0" layer="19" extent="1-1"/>
 </signal>
 <signal name="SCL">
@@
 </polygon>
 <polygon width="0.1524" layer="16" thermals="no" rank="2">
-<vertex x="68.961" y="81.026"/>
+<vertex x="68.961" y="79.883"/>
 <vertex x="68.961" y="82.55" curve="-90"/>
-<vertex x="69.723" y="83.312"/>
-<vertex x="74.168" y="83.312" curve="90"/>
-<vertex x="74.93" y="84.074"/>
-<vertex x="74.93" y="86.995" curve="-90"/>
-<vertex x="75.438" y="87.503"/>
-<vertex x="86.868" y="79.883" curve="-90"/>
-<vertex x="87.884" y="78.867"/>
-<vertex x="87.884" y="77.47" curve="-90"/>
 <vertex x="76.708" y="79.248" curve="90"/>
-<vertex x="76.327" y="79.629"/>
-<vertex x="71.882" y="79.629"/>
 <vertex x="69.215" y="79.629" curve="-90"/>
-<vertex x="68.961" y="79.883"/>
-</polygon>
-</signal>
+</polygon>
+</signal>

Commit message: Cganges
Parts:
- removed Q1, Q2: 2N7002-7-F, SamacSys_Parts:SOT96P240X120-3N
- removed Q5: SQJ912AEP-T2_BE3, SamacSys_Parts:SQJ968EPT1_GE3
- removed Q7: SI7923DN-T1-E3, SamacSys_Parts:POWERPAK-1212-8_DUAL
- removed R10: ERJ-D2DFR022V, SamacSys_Parts:RESC3216X80N
- removed R13, R14, R15, R16, R3, R5, R9: 1k, SamacSys_Parts:RESC1608X55N
- added IC3: MC33HB2000AES, SamacSys_Parts:MC33HB2000AES
- C24: value 0.1uF -> 1uF
- moved C24 15.0 mm to (76.3, 81.7), turned to 90 degrees
- moved C21 0.89 mm to (48.9, 73.2)
Connections:
- removed net FWD: Q1.3, Q7.4, R14.1
- removed net N$13: Q1.1, R16.1
- removed net N$2: Q5.2, R3.1
- removed net N$4: Q2.1, R15.1
- removed net RVRS: Q2.3, Q7.2, R13.1
- removed net SRC: Q5.1, Q5.3, R10.2, R9.2
- new net CS: IC3.27, IC4.63
- new net DISABLE: IC3.7, IC4.18
- new net ENABLE: IC3.6, IC4.19
- new net MISO: IC3.1, IC4.15
- new net MOSI: IC3.3, IC4.13
- new net N$12: IC3.16, IC3.17, IC3.18, IC3.19
- new net N$18: C24.2, IC3.26
- new net SCLK: IC3.2, IC4.14
- net 0: now also IC3.20, IC3.21, IC3.4, IC3.5; no longer C24.2, Q1.2, Q2.2, R10.1
- net D1: now also IC3.13, IC3.14; no longer Q5.5, Q5.7, Q5.9, Q7.7, Q7.8
- net D2: now also IC3.22, IC3.23; no longer Q5.10, Q5.6, Q5.8, Q7.5, Q7.6
- net FORWARD: now also IC3.8; no longer R15.2, R3.2
- net IMOTOR: now also IC3.10; no longer C24.1, R9.1
- net N$7: now also IC3.29, IC3.30, IC3.31, IC3.32, IC3.33, IC3.34, IC3.35, IC3.36, IC3.37; no longer Q5.4, R5.1
- net REVERSE: now also IC3.9; no longer R16.2, R5.2
- net VBUS: now also C24.1, IC3.11, IC3.12, IC3.24, IC3.25; no longer Q7.1, Q7.3, R13.2, R14.2
- net VDD: now also IC3.28
Routing:
- net CS: track 0.00 -> 40.9 mm, vias 0 -> 4
- net ENABLE: track 0.00 -> 32.3 mm, vias 0 -> 2
- net MOSI: track 0.00 -> 31.5 mm, vias 0 -> 2
- net DISABLE: track 0.00 -> 30.5 mm, vias 0 -> 2
- net MISO: track 0.00 -> 28.4 mm, vias 0 -> 2
- net SCLK: track 0.00 -> 26.7 mm, vias 0 -> 2
- net VDD: track 96.1 -> 118.1 mm, vias 8 -> 10
- net RVRS: track 16.2 -> 0.00 mm
- net FWD: track 13.8 -> 0.00 mm
- net N$7: track 13.4 -> 0.00 mm, vias 2 -> 0
- net N$18: track 0.00 -> 11.5 mm, vias 0 -> 2
- net VBUS: track 10.4 -> 19.0 mm, vias 4 -> 6
- net N$13: track 8.44 -> 0.00 mm
- net N$4: track 8.33 -> 0.00 mm
- net REVERSE: track 19.6 -> 27.5 mm
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- removed copper zone on layer 16, net 5V
- removed copper zone on layer 16, net D1
- removed copper zone on layer 1, net SRC

Commit message: Changes
Connections:
- removed net N$12: IC3.16, IC3.17, IC3.18, IC3.19
- removed net N$7: IC3.29, IC3.30, IC3.31, IC3.32, IC3.33, IC3.34, IC3.35, IC3.36, IC3.37
- net 0: now also IC3.16, IC3.17, IC3.18, IC3.19, IC3.29, IC3.30, IC3.31, IC3.32, IC3.33, IC3.34, IC3.35, IC3.36, IC3.37
Routing:
- net CS: track 40.9 -> 41.4 mm
